File: IOB-I2C-MCP23017.sch (EAGLE design)
At the start: 10 parts, among them IC1 MCP23017SO

Commit message: cleanup layout
Parts:
- removed U$5: I2C-EXPANDER, SPCoast:I2C-EXPANDER
- added BOARD: CONNECTOR-I2C-EXPANDER, SPCoast:CONNECTOR-I2C-EXPANDER
- LED1: value (none) -> G
- R4: value 2k2 -> 4k7
Connections:
- net GND: now also BOARD.GND; no longer U$5.GND
- net P1: now also BOARD.IO1; no longer U$5.IO1
- net P10: now also BOARD.IO10; no longer U$5.IO10
- net P11: now also BOARD.IO11; no longer U$5.IO11
- net P12: now also BOARD.IO12; no longer U$5.IO12
- net P13: now also BOARD.IO13; no longer U$5.IO13
- net P14: now also BOARD.IO14; no longer U$5.IO14
- net P15: now also BOARD.IO15; no longer U$5.IO15
- net P16: now also BOARD.IO16; no longer U$5.IO16
- net P2: now also BOARD.IO2; no longer U$5.IO2
- net P3: now also BOARD.IO3; no longer U$5.IO3
- net P4: now also BOARD.IO4; no longer U$5.IO4
- net P5: now also BOARD.IO5; no longer U$5.IO5
- net P6: now also BOARD.IO6; no longer U$5.IO6
- net P7: now also BOARD.IO7; no longer U$5.IO7
- net P8: now also BOARD.IO8; no longer U$5.IO8
- net P9: now also BOARD.IO9; no longer U$5.IO9
- net SCL: now also BOARD.SCL; no longer U$5.SCL
- net SDA: now also BOARD.SDA; no longer U$5.SDA
- net VCC: now also BOARD.VCC; no longer U$5.VCC
Changed lines of the file:
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@@
 <part name="P+24" library="supply1" deviceset="VCC" device=""/>
 <part name="GND5" library="SPCoast" deviceset="GND" device=""/>
-<part name="U$5" library="SPCoast" deviceset="I2C-EXPANDER" device=""/>
+<part name="BOARD" library="SPCoast" deviceset="CONNECTOR-I2C-EXPANDER" device=""/>
 <part name="C1" library="SPCoast" deviceset="CAP*" device="0603" value="0.1uF"/>
 <part name="P+1" library="supply1" deviceset="VCC" device=""/>
 <part name="GND1" library="SPCoast" deviceset="GND" device=""/>
-<part name="LED1" library="SPCoast" deviceset="LED*" device="0805-LED"/>
-<part name="R4" library="SPCoast" deviceset="R*" device="0603-RES" value="2k2"/>
+<part name="LED1" library="SPCoast" deviceset="LED*" device="0805-LED" value="G"/>
+<part name="R4" library="SPCoast" deviceset="R*" device="0603-RES" value="4k7"/>
 <part name="P+2" library="supply1" deviceset="VCC" device=""/>
 </parts>
@@
 </instance>
 <instance part="GND5" gate="1" x="109.22" y="99.06"/>
-<instance part="U$5" gate="G$1" x="180.34" y="124.46"/>
+<instance part="BOARD" gate="G$1" x="180.34" y="124.46"/>
 <instance part="C1" gate="C1" x="78.74" y="149.86"/>
 <instance part="P+1" gate="VCC" x="78.74" y="154.94" smashed="yes" rot="MR0">
@@
 </segment>
 <segment>
-<pinref part="U$5" gate="G$1" pin="GND"/>
+<pinref part="BOARD" gate="G$1" pin="GND"/>
 <pinref part="GND3" gate="1" pin="GND"/>
 </segment>
@@
 </segment>
 <segment>
-<pinref part="U$5" gate="G$1" pin="IO1"/>
+<pinref part="BOARD" gate="G$1" pin="IO1"/>
 <wire x1="167.64" y1="134.62" x2="165.1" y2="134.62" width="0.1524" layer="91"/>
 <label x="165.1" y="134.62" size="1.016" layer="95" rot="R180" xref="yes"/>
@@
 </segment>
 <segment>
-<pinref part="U$5" gate="G$1" pin="IO2"/>
+<pinref part="BOARD" gate="G$1" pin="IO2"/>
 <wire x1="167.64" y1="132.08" x2="165.1" y2="132.08" width="0.1524" layer="91"/>
 <label x="165.1" y="132.08" size="1.016" layer="95" rot="R180" xref="yes"/>
@@
 </segment>
 <segment>
-<pinref part="U$5" gate="G$1" pin="IO3"/>
+<pinref part="BOARD" gate="G$1" pin="IO3"/>
 <wire x1="167.64" y1="129.54" x2="165.1" y2="129.54" width="0.1524" layer="91"/>
 <label x="165.1" y="129.54" size="1.016" layer="95" rot="R180" xref="yes"/>
@@
 </segment>
 <segment>
-<pinref part="U$5" gate="G$1" pin="IO4"/>
+<pinref part="BOARD" gate="G$1" pin="IO4"/>
 <wire x1="167.64" y1="127" x2="165.1" y2="127" width="0.1524" layer="91"/>
 <label x="165.1" y="127" size="1.016" layer="95" rot="R180" xref="yes"/>
@@
 </segment>
 <segment>
-<pinref part="U$5" gate="G$1" pin="IO5"/>
+<pinref part="BOARD" gate="G$1" pin="IO5"/>
 <wire x1="167.64" y1="124.46" x2="165.1" y2="124.46" width="0.1524" layer="91"/>
 <label x="165.1" y="124.46" size="1.016" layer="95" rot="R180" xref="yes"/>
@@
 </segment>
 <segment>
-<pinref part="U$5" gate="G$1" pin="IO6"/>
+<pinref part="BOARD" gate="G$1" pin="IO6"/>
 <wire x1="167.64" y1="121.92" x2="165.1" y2="121.92" width="0.1524" layer="91"/>
 <label x="165.1" y="121.92" size="1.016" layer="95" rot="R180" xref="yes"/>
@@
 </segment>
 <segment>
-<pinref part="U$5" gate="G$1" pin="IO7"/>
+<pinref part="BOARD" gate="G$1" pin="IO7"/>
 <wire x1="167.64" y1="119.38" x2="165.1" y2="119.38" width="0.1524" layer="91"/>
 <label x="165.1" y="119.38" size="1.016" layer="95" rot="R180" xref="yes"/>
@@
 </segment>
 <segment>
-<pinref part="U$5" gate="G$1" pin="IO8"/>
+<pinref part="BOARD" gate="G$1" pin="IO8"/>
 <wire x1="167.64" y1="116.84" x2="165.1" y2="116.84" width="0.1524" layer="91"/>
 <label x="165.1" y="116.84" size="1.016" layer="95" rot="R180" xref="yes"/>
@@
 </segment>
 <segment>
-<pinref part="U$5" gate="G$1" pin="IO13"/>
+<pinref part="BOARD" gate="G$1" pin="IO13"/>
 <wire x1="193.04" y1="124.46" x2="195.58" y2="124.46" width="0.1524" layer="91"/>
 <label x="195.58" y="124.46" size="1.016" layer="95" xref="yes"/>
@@
 </segment>
 <segment>
-<pinref part="U$5" gate="G$1" pin="IO14"/>
+<pinref part="BOARD" gate="G$1" pin="IO14"/>
 <wire x1="193.04" y1="121.92" x2="195.58" y2="121.92" width="0.1524" layer="91"/>
 <label x="195.58" y="121.92" size="1.016" layer="95" xref="yes"/>
@@
 </segment>
 <segment>
-<pinref part="U$5" gate="G$1" pin="IO15"/>
+<pinref part="BOARD" gate="G$1" pin="IO15"/>
 <wire x1="193.04" y1="119.38" x2="195.58" y2="119.38" width="0.1524" layer="91"/>
 <label x="195.58" y="119.38" size="1.016" layer="95" xref="yes"/>
@@
 </segment>
 <segment>
-<pinref part="U$5" gate="G$1" pin="IO16"/>
+<pinref part="BOARD" gate="G$1" pin="IO16"/>
 <wire x1="193.04" y1="116.84" x2="195.58" y2="116.84" width="0.1524" layer="91"/>
 <label x="195.58" y="116.84" size="1.016" layer="95" xref="yes"/>
@@
 </segment>
 <segment>
-<pinref part="U$5" gate="G$1" pin="VCC"/>
+<pinref part="BOARD" gate="G$1" pin="VCC"/>
 <pinref part="P+4" gate="VCC" pin="VCC"/>
 </segment>
@@
 </segment>
 <segment>
-<pinref part="U$5" gate="G$1" pin="SDA"/>
+<pinref part="BOARD" gate="G$1" pin="SDA"/>
 <wire x1="193.04" y1="114.3" x2="198.12" y2="114.3" width="0.1524" layer="91"/>
 <label x="198.12" y="114.3" size="1.016" layer="95" xref="yes"/>
@@
 </segment>
 <segment>
-<pinref part="U$5" gate="G$1" pin="SCL"/>
+<pinref part="BOARD" gate="G$1" pin="SCL"/>
 <wire x1="193.04" y1="111.76" x2="198.12" y2="111.76" width="0.1524" layer="91"/>
 <label x="198.12" y="111.76" size="1.016" layer="95" xref="yes"/>
@@
 </segment>
 <segment>
-<pinref part="U$5" gate="G$1" pin="IO9"/>
+<pinref part="BOARD" gate="G$1" pin="IO9"/>
 <wire x1="193.04" y1="134.62" x2="195.58" y2="134.62" width="0.1524" layer="91"/>
 <label x="195.58" y="134.62" size="1.016" layer="95" xref="yes"/>
@@
 </segment>
 <segment>
-<pinref part="U$5" gate="G$1" pin="IO10"/>
+<pinref part="BOARD" gate="G$1" pin="IO10"/>
 <wire x1="193.04" y1="132.08" x2="195.58" y2="132.08" width="0.1524" layer="91"/>
 <label x="195.58" y="132.08" size="1.016" layer="95" xref="yes"/>
@@
 </segment>
 <segment>
-<pinref part="U$5" gate="G$1" pin="IO11"/>
+<pinref part="BOARD" gate="G$1" pin="IO11"/>
 <wire x1="193.04" y1="129.54" x2="195.58" y2="129.54" width="0.1524" layer="91"/>
 <label x="195.58" y="129.54" size="1.016" layer="95" xref="yes"/>
@@
 </segment>
 <segment>
-<pinref part="U$5" gate="G$1" pin="IO12"/>
+<pinref part="BOARD" gate="G$1" pin="IO12"/>
 <wire x1="193.04" y1="127" x2="195.58" y2="127" width="0.1524" layer="91"/>
 <label x="195.58" y="127" size="1.016" layer="95" xref="yes"/>

Commit message: added missing values
Parts:
- SW1: value (none) -> SPSTx4
Changed lines of the file:
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@@
 <part name="IC1" library="microchip" deviceset="MCP23017" device="SO"/>
 <part name="GND3" library="SPCoast" deviceset="GND" device=""/>
-<part name="SW1" library="SPCoast" deviceset="SW_DIP-4" device=""/>
+<part name="SW1" library="SPCoast" deviceset="SW_DIP-4" device="" value="SPSTx4"/>
 <part name="R1" library="SPCoast" deviceset="R*" device="0603-RES" value="10K"/>
 <part name="R2" library="SPCoast" deviceset="R*" device="0603-RES" value="10K"/>

Commit message: normalized values
Parts:
- LED1: device SPCoast:LED0805-LED -> SPCoast:LED0603-LED
- OSHW1: value DOC-OSHW-LOGO-M -> OSHW
Changed lines of the file:
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@@
 <parts>
 <part name="FRAME1" library="SPCoast" deviceset="DOC-FRAME-LETTER" device=""/>
-<part name="OSHW1" library="SPCoast" deviceset="DOC-OSHW-LOGO-" device="M"/>
+<part name="OSHW1" library="SPCoast" deviceset="DOC-OSHW-LOGO-" device="M" value="OSHW"/>
 <part name="IC1" library="microchip" deviceset="MCP23017" device="SO"/>
 <part name="GND3" library="SPCoast" deviceset="GND" device=""/>
@@
 <part name="P+1" library="supply1" deviceset="VCC" device=""/>
 <part name="GND1" library="SPCoast" deviceset="GND" device=""/>
-<part name="LED1" library="SPCoast" deviceset="LED*" device="0805-LED" value="G"/>
+<part name="LED1" library="SPCoast" deviceset="LED*" device="0603-LED" value="G"/>
 <part name="R4" library="SPCoast" deviceset="R*" device="0603-RES" value="4k7"/>
 <part name="P+2" library="supply1" deviceset="VCC" device=""/>
