File: IOB-I2C-MCP23017_array.brd (EAGLE design)
At the start: 108.7 x 112 mm, 33 parts, among them IC1X11 MCP23017SO, IC1X12 MCP23017SO, IC1X13 MCP23017SO

Commit message: cleanup
Other:
- board text added: "Input Changed"
Changed lines of the file:
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@@
 <layer number="23" name="tOrigins" color="15" fill="1" visible="yes" active="yes"/>
 <layer number="24" name="bOrigins" color="15" fill="1" visible="no" active="yes"/>
-<layer number="25" name="tNames" color="7" fill="1" visible="no" active="yes"/>
+<layer number="25" name="tNames" color="7" fill="1" visible="yes" active="yes"/>
 <layer number="26" name="bNames" color="7" fill="1" visible="no" active="yes"/>
-<layer number="27" name="tValues" color="7" fill="1" visible="no" active="yes"/>
+<layer number="27" name="tValues" color="7" fill="1" visible="yes" active="yes"/>
 <layer number="28" name="bValues" color="7" fill="1" visible="no" active="yes"/>
 <layer number="29" name="tStop" color="7" fill="3" visible="no" active="yes"/>
@@
 <layer number="45" name="Holes" color="7" fill="1" visible="yes" active="yes"/>
 <layer number="46" name="Milling" color="3" fill="1" visible="yes" active="yes"/>
-<layer number="47" name="Measures" color="7" fill="1" visible="no" active="yes"/>
+<layer number="47" name="Measures" color="7" fill="1" visible="yes" active="yes"/>
 <layer number="48" name="Document" color="7" fill="1" visible="yes" active="yes"/>
 <layer number="49" name="Reference" color="7" fill="1" visible="yes" active="yes"/>
@@
 <layer number="99" name="Anatomie" color="7" fill="1" visible="no" active="no"/>
 <layer number="100" name="Muster" color="7" fill="1" visible="no" active="no"/>
-<layer number="101" name="Hidden" color="57" fill="4" visible="no" active="yes"/>
-<layer number="102" name="Changes" color="13" fill="1" visible="no" active="yes"/>
+<layer number="101" name="Hidden" color="57" fill="4" visible="yes" active="yes"/>
+<layer number="102" name="Changes" color="13" fill="1" visible="yes" active="yes"/>
 <layer number="103" name="tMap" color="29" fill="4" visible="no" active="yes"/>
-<layer number="104" name="Name" color="16" fill="1" visible="no" active="yes"/>
+<layer number="104" name="Name" color="16" fill="1" visible="yes" active="yes"/>
 <layer number="105" name="tPlate" color="7" fill="1" visible="no" active="yes"/>
 <layer number="106" name="bPlate" color="7" fill="1" visible="no" active="yes"/>
@@
 <plain>
 <text x="34.29" y="13.335" size="0.6096" layer="19" font="vector" ratio="10">C1</text>
-<text x="49.53" y="26.035" size="1.27" layer="19" font="vector" ratio="10" rot="R180">LED1</text>
 <text x="46.99" y="31.115" size="0.8128" layer="19" font="vector" ratio="10">R4</text>
 <wire x1="12.7" y1="33.02" x2="12.7" y2="0" width="0" layer="101"/>
@@
 <wire x1="72.39" y1="16.51" x2="72.39" y2="1.27" width="2.1844" layer="22"/>
 <wire x1="80.01" y1="16.51" x2="80.01" y2="1.27" width="2.1844" layer="22"/>
+<wire x1="48.26" y1="15.24" x2="48.26" y2="19.05" width="0.4064" layer="21"/>
+<wire x1="48.26" y1="19.05" x2="49.53" y2="17.78" width="0.4064" layer="21"/>
+<wire x1="48.26" y1="19.05" x2="46.99" y2="17.78" width="0.4064" layer="21"/>
 <text x="35.56" y="30.48" size="1.9304" layer="21" font="vector" ratio="10">IOB-I2C-MCP23017</text>
 <text x="60.96" y="1.524" size="1.016" layer="21" font="vector" ratio="10">2020-09</text>
@@
 <text x="62.5" y="12.827" size="1.4224" layer="22" font="vector" ratio="15" rot="MR300">Go Bears!</text>
 <text x="34.29" y="13.335" size="0.6096" layer="125" font="vector">C1</text>
-<text x="40.894" y="26.924" size="1.778" layer="125" font="vector" ratio="10">IC1</text>
-<text x="49.53" y="26.035" size="1.27" layer="125" font="vector" rot="R180">LED1</text>
+<text x="50.546" y="20.574" size="1.778" layer="125" font="vector" ratio="10" rot="R90">IC1</text>
+<text x="55.88" y="27.305" size="1.27" layer="125" font="vector" rot="R180">LED1</text>
 <text x="55.499" y="7.62" size="0.8128" layer="125" font="vector" rot="R270">R1</text>
 <text x="63.246" y="9.652" size="0.8128" layer="125" font="vector" rot="R90">R2</text>
@@
 <text x="11.938" y="30.861" size="0.4064" layer="204" font="vector" rot="R270">U$5</text>
 <text x="62.738" y="30.861" size="0.4064" layer="204" font="vector" rot="R270">U$5</text>
-<text x="34.29" y="46.355" size="0.6096" layer="19" font="vector">C1</text>
-<text x="49.53" y="59.055" size="1.27" layer="19" font="vector" rot="R180">LED1</text>
-<text x="46.99" y="64.135" size="0.8128" layer="19" font="vector">R4</text>
+<text x="40.767" y="26.289" size="0.8128" layer="21">Input
+Changed</text>
+<text x="34.29" y="46.355" size="0.6096" layer="19">C1</text>
+<text x="46.99" y="64.135" size="0.8128" layer="19">R4</text>
 <wire x1="12.7" y1="66.04" x2="12.7" y2="33.02" width="0" layer="101"/>
 <wire x1="12.7" y1="33.02" x2="83.82" y2="33.02" width="0" layer="101"/>
@@
 <wire x1="72.39" y1="49.53" x2="72.39" y2="34.29" width="2.1844" layer="22"/>
 <wire x1="80.01" y1="49.53" x2="80.01" y2="34.29" width="2.1844" layer="22"/>
+<wire x1="48.26" y1="48.26" x2="48.26" y2="52.07" width="0.4064" layer="21"/>
+<wire x1="48.26" y1="52.07" x2="49.53" y2="50.8" width="0.4064" layer="21"/>
+<wire x1="48.26" y1="52.07" x2="46.99" y2="50.8" width="0.4064" layer="21"/>
 <text x="35.56" y="63.5" size="1.9304" layer="21" font="vector" ratio="10">IOB-I2C-MCP23017</text>
 <text x="60.96" y="34.544" size="1.016" layer="21" font="vector" ratio="10">2020-09</text>
@@
 <text x="62.5" y="45.847" size="1.4224" layer="22" font="vector" ratio="15" rot="MR300">Go Bears!</text>
 <text x="34.29" y="46.355" size="0.6096" layer="125" font="vector">C1</text>
-<text x="40.894" y="59.944" size="1.778" layer="125" font="vector" ratio="10">IC1</text>
-<text x="49.53" y="59.055" size="1.27" layer="125" font="vector" rot="R180">LED1</text>
+<text x="50.546" y="53.594" size="1.778" layer="125" font="vector" ratio="10" rot="R90">IC1</text>
+<text x="55.88" y="60.325" size="1.27" layer="125" font="vector" rot="R180">LED1</text>
 <text x="55.499" y="40.64" size="0.8128" layer="125" font="vector" rot="R270">R1</text>
 <text x="63.246" y="42.672" size="0.8128" layer="125" font="vector" rot="R90">R2</text>
@@
 <text x="11.938" y="63.881" size="0.4064" layer="204" font="vector" rot="R270">U$5</text>
 <text x="62.738" y="63.881" size="0.4064" layer="204" font="vector" rot="R270">U$5</text>
-<wire x1="12.7" y1="0" x2="83.82" y2="0" width="0.254" layer="20"/>
-<wire x1="83.82" y1="0" x2="83.82" y2="99.06" width="0.254" layer="20"/>
-<wire x1="83.82" y1="99.06" x2="12.7" y2="99.06" width="0.254" layer="20"/>
-<wire x1="12.7" y1="99.06" x2="12.7" y2="0" width="0.254" layer="20"/>
-<text x="34.29" y="79.375" size="0.6096" layer="19" font="vector">C1</text>
-<text x="49.53" y="92.075" size="1.27" layer="19" font="vector" rot="R180">LED1</text>
-<text x="46.99" y="97.155" size="0.8128" layer="19" font="vector">R4</text>
+<text x="40.767" y="59.309" size="0.8128" layer="21">Input
+Changed</text>
+<text x="34.29" y="79.375" size="0.6096" layer="19">C1</text>
+<text x="46.99" y="97.155" size="0.8128" layer="19">R4</text>
 <wire x1="12.7" y1="99.06" x2="12.7" y2="66.04" width="0" layer="101"/>
 <wire x1="12.7" y1="66.04" x2="83.82" y2="66.04" width="0" layer="101"/>
@@
 <wire x1="72.39" y1="82.55" x2="72.39" y2="67.31" width="2.1844" layer="22"/>
 <wire x1="80.01" y1="82.55" x2="80.01" y2="67.31" width="2.1844" layer="22"/>
+<wire x1="48.26" y1="81.28" x2="48.26" y2="85.09" width="0.4064" layer="21"/>
+<wire x1="48.26" y1="85.09" x2="49.53" y2="83.82" width="0.4064" layer="21"/>
+<wire x1="48.26" y1="85.09" x2="46.99" y2="83.82" width="0.4064" layer="21"/>
 <text x="35.56" y="96.52" size="1.9304" layer="21" font="vector" ratio="10">IOB-I2C-MCP23017</text>
 <text x="60.96" y="67.564" size="1.016" layer="21" font="vector" ratio="10">2020-09</text>
@@
 <text x="62.5" y="78.867" size="1.4224" layer="22" font="vector" ratio="15" rot="MR300">Go Bears!</text>
 <text x="34.29" y="79.375" size="0.6096" layer="125" font="vector">C1</text>
-<text x="40.894" y="92.964" size="1.778" layer="125" font="vector" ratio="10">IC1</text>
-<text x="49.53" y="92.075" size="1.27" layer="125" font="vector" rot="R180">LED1</text>
+<text x="50.546" y="86.614" size="1.778" layer="125" font="vector" ratio="10" rot="R90">IC1</text>
+<text x="55.88" y="93.345" size="1.27" layer="125" font="vector" rot="R180">LED1</text>
 <text x="55.499" y="73.66" size="0.8128" layer="125" font="vector" rot="R270">R1</text>
 <text x="63.246" y="75.692" size="0.8128" layer="125" font="vector" rot="R90">R2</text>
@@
 <text x="11.938" y="96.901" size="0.4064" layer="204" font="vector" rot="R270">U$5</text>
 <text x="62.738" y="96.901" size="0.4064" layer="204" font="vector" rot="R270">U$5</text>
+<text x="40.767" y="92.329" size="0.8128" layer="21">Input
+Changed</text>
 <text x="9.271" y="47.498" size="1.27" layer="21" font="vector" ratio="10" rot="R90">v1.0</text>
 </plain>
@@
 </board>
 </drawing>
+<compatibility>
+<note version="6.3" minversion="6.2.2" severity="warning">
+Since Version 6.2.2 text objects can contain more than one line,
+which will not be processed correctly with this version.
+</note>
+</compatibility>
 </eagle>

Commit message: cleanup layout
Parts:
- BOARDX11, BOARDX12, BOARDX13: value I2C-EXPANDER -> CONNECTOR-I2C-EXPANDER
- LED1X11, LED1X12, LED1X13: value (none) -> G
- R4X11, R4X12, R4X13: value 2k2 -> 4k7
- moved R4X12 4.49 mm to (44.2, 61.0), turned to 180 degrees
- moved R4X13 4.49 mm to (44.2, 94.0), turned to 180 degrees
- moved R4X11 4.49 mm to (44.2, 27.9), turned to 180 degrees
- moved SW1X11 1.27 mm to (72.4, 14.0)
- moved SW1X12 1.27 mm to (72.4, 47.0)
- moved SW1X13 1.27 mm to (72.4, 80.0)
- moved LED1X13 0.64 mm to (48.3, 94.0)
- moved LED1X11 0.64 mm to (48.3, 27.9)
- moved LED1X12 0.63 mm to (48.3, 61.0)
- moved OSHW1X12 0.40 mm to (47.8, 37.2)
- moved OSHW1X13 0.40 mm to (47.8, 70.2)
- moved OSHW1X11 0.40 mm to (47.8, 4.19)
- renumbered U$5X11 to BOARDX11, U$5X12 to BOARDX12, U$5X13 to BOARDX13
Routing:
- net SDAX12: track 51.3 -> 78.1 mm, vias 1 -> 3
- net SDAX11: track 51.3 -> 78.1 mm, vias 1 -> 3
- net SDAX13: track 51.3 -> 78.1 mm, vias 1 -> 3
- net SCLX12: track 75.6 -> 79.5 mm
- net SCLX13: track 75.6 -> 79.5 mm
- net SCLX11: track 75.6 -> 79.5 mm
- net A1X12: track 39.3 -> 36.8 mm
- net A1X11: track 39.3 -> 36.8 mm
- net A1X13: track 39.3 -> 36.8 mm
- net P4X13: track 25.7 -> 24.2 mm
- net P4X12: track 25.7 -> 24.2 mm
- net P4X11: track 25.7 -> 24.2 mm
- net A3X13: track 24.0 -> 22.7 mm
- net A0X12: track 29.1 -> 27.9 mm
- net A0X11: track 29.1 -> 27.9 mm
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Other:
- board text added: "BOARD"
- board text added: "I2C Address"
- board text added: "MCP23017SO"
- board text added: "SO28-W"
- board text removed: "Address"
- board text removed: "Board I2C"
- board text removed: "U$5"

Commit message: added values for connectors
Parts:
- FID_LR, FID_UL: value (none) -> FIDUCIAL
- U$5X1: value (none) -> 10x10
Changed lines of the file:
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@@
 <attribute name="VALUE" x="78.232" y="86.614" size="0.8128" layer="27" ratio="10" rot="R180"/>
 </element>
-<element name="U$5X1" library="SPCoast" package="BOARD-TEMPLATE-IOB-I2C-3X1-ARRAY" value="" x="0" y="0"/>
-<element name="FID_UL" library="SPCoast" package="FIDUCIAL_1MM" value="" x="5.08" y="91.44"/>
-<element name="FID_LR" library="SPCoast" package="FIDUCIAL_1MM" value="" x="93.98" y="8.89"/>
+<element name="U$5X1" library="SPCoast" package="BOARD-TEMPLATE-IOB-I2C-3X1-ARRAY" value="10x10" x="0" y="0"/>
+<element name="FID_UL" library="SPCoast" package="FIDUCIAL_1MM" value="FIDUCIAL" x="5.08" y="91.44"/>
+<element name="FID_LR" library="SPCoast" package="FIDUCIAL_1MM" value="FIDUCIAL" x="93.98" y="8.89"/>
 </elements>
 <signals>

Commit message: added missing values
Parts:
- SW1X11, SW1X12, SW1X13: value (none) -> SPSTx4
Changed lines of the file:
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@@
 <attribute name="VALUE" x="45.466" y="29.845" size="0.8128" layer="27" font="vector" rot="R180"/>
 </element>
-<element name="SW1X11" library="SPCoast" package="EDG-04" value="" x="72.39" y="13.97" smashed="yes" rot="R180">
+<element name="SW1X11" library="SPCoast" package="EDG-04" value="SPSTx4" x="72.39" y="13.97" smashed="yes" rot="R180">
 <attribute name="VALUE" x="78.232" y="20.574" size="0.8128" layer="27" ratio="10" rot="R180"/>
 </element>
@@
 <attribute name="VALUE" x="45.466" y="62.865" size="0.8128" layer="27" font="vector" rot="R180"/>
 </element>
-<element name="SW1X12" library="SPCoast" package="EDG-04" value="" x="72.39" y="46.99" smashed="yes" rot="R180">
+<element name="SW1X12" library="SPCoast" package="EDG-04" value="SPSTx4" x="72.39" y="46.99" smashed="yes" rot="R180">
 <attribute name="VALUE" x="78.232" y="53.594" size="0.8128" layer="27" ratio="10" rot="R180"/>
 </element>
@@
 <attribute name="VALUE" x="45.466" y="95.885" size="0.8128" layer="27" font="vector" rot="R180"/>
 </element>
-<element name="SW1X13" library="SPCoast" package="EDG-04" value="" x="72.39" y="80.01" smashed="yes" rot="R180">
+<element name="SW1X13" library="SPCoast" package="EDG-04" value="SPSTx4" x="72.39" y="80.01" smashed="yes" rot="R180">
 <attribute name="VALUE" x="78.232" y="86.614" size="0.8128" layer="27" ratio="10" rot="R180"/>
 </element>

Commit message: normalized values
Parts:
- LED1X11, LED1X12, LED1X13: device SPCoast:0805-LED -> SPCoast:0603-LED
- U$5X1: value 10x10 -> BOARD
Changed lines of the file:
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@@
 </element>
 <element name="IC1X11" library="microchip" package="SO28W" value="MCP23017SO" x="47.498" y="17.145" smashed="yes" rot="R270"/>
-<element name="LED1X11" library="SPCoast" package="0805-LED" value="G" x="48.26" y="27.94" smashed="yes" rot="R180">
+<element name="LED1X11" library="SPCoast" package="0603-LED" value="G" x="48.26" y="27.94" smashed="yes" rot="R180">
 <attribute name="VALUE" x="49.53" y="30.48" size="1.27" layer="27" rot="R180"/>
 </element>
@@
 </element>
 <element name="IC1X12" library="microchip" package="SO28W" value="MCP23017SO" x="47.498" y="50.165" smashed="yes" rot="R270"/>
-<element name="LED1X12" library="SPCoast" package="0805-LED" value="G" x="48.26" y="60.96" smashed="yes" rot="R180">
+<element name="LED1X12" library="SPCoast" package="0603-LED" value="G" x="48.26" y="60.96" smashed="yes" rot="R180">
 <attribute name="VALUE" x="49.53" y="63.5" size="1.27" layer="27" rot="R180"/>
 </element>
@@
 </element>
 <element name="IC1X13" library="microchip" package="SO28W" value="MCP23017SO" x="47.498" y="83.185" smashed="yes" rot="R270"/>
-<element name="LED1X13" library="SPCoast" package="0805-LED" value="G" x="48.26" y="93.98" smashed="yes" rot="R180">
+<element name="LED1X13" library="SPCoast" package="0603-LED" value="G" x="48.26" y="93.98" smashed="yes" rot="R180">
 <attribute name="VALUE" x="49.53" y="96.52" size="1.27" layer="27" rot="R180"/>
 </element>
@@
 <attribute name="VALUE" x="78.232" y="86.614" size="0.8128" layer="27" ratio="10" rot="R180"/>
 </element>
-<element name="U$5X1" library="SPCoast" package="BOARD-TEMPLATE-IOB-I2C-3X1-ARRAY" value="10x10" x="0" y="0"/>
+<element name="U$5X1" library="SPCoast" package="BOARD-TEMPLATE-IOB-I2C-3X1-ARRAY" value="BOARD" x="0" y="0"/>
 <element name="FID_UL" library="SPCoast" package="FIDUCIAL_1MM" value="FIDUCIAL" x="5.08" y="91.44"/>
 <element name="FID_LR" library="SPCoast" package="FIDUCIAL_1MM" value="FIDUCIAL" x="93.98" y="8.89"/>
@@
 <signal name="A0X11">
 <wire x1="52.278" y1="8.255" x2="55.88" y2="8.255" width="0.254" layer="1"/>
-<wire x1="57.15" y1="7.2" x2="55.88" y2="8.255" width="0.254" layer="1"/>
+<wire x1="57.15" y1="7.239" x2="55.88" y2="8.255" width="0.254" layer="1"/>
 <wire x1="59.69" y1="5.715" x2="73.66" y2="5.715" width="0.254" layer="1"/>
 <wire x1="73.66" y1="5.715" x2="76.2" y2="8.255" width="0.254" layer="1"/>
@@
 <wire x1="59.69" y1="5.715" x2="58.42" y2="6.985" width="0.254" layer="1"/>
 <wire x1="58.42" y1="6.985" x2="57.365" y2="6.985" width="0.254" layer="1"/>
-<wire x1="57.365" y1="6.985" x2="57.15" y2="7.2" width="0.254" layer="1"/>
+<wire x1="57.365" y1="6.985" x2="57.15" y2="7.239" width="0.254" layer="1"/>
 <contactref element="SW1X11" pad="8"/>
 <contactref element="IC1X11" pad="15"/>
@@
 <wire x1="72.39" y1="6.985" x2="73.66" y2="8.255" width="0.254" layer="1"/>
 <wire x1="73.66" y1="8.255" x2="73.66" y2="11.43" width="0.254" layer="1"/>
-<wire x1="64.135" y1="9.945" x2="65.19" y2="9.945" width="0.254" layer="1"/>
+<wire x1="64.135" y1="9.906" x2="65.19" y2="9.945" width="0.254" layer="1"/>
 <wire x1="65.19" y1="9.945" x2="67.31" y2="12.065" width="0.254" layer="1"/>
 <wire x1="67.31" y1="12.065" x2="73.025" y2="12.065" width="0.254" layer="1"/>
@@
 <wire x1="69.85" y1="8.255" x2="71.12" y2="9.525" width="0.254" layer="1"/>
 <wire x1="71.12" y1="9.525" x2="71.12" y2="10.16" width="0.254" layer="1"/>
-<wire x1="60.96" y1="9.945" x2="60.96" y2="8.255" width="0.254" layer="1"/>
+<wire x1="60.96" y1="9.906" x2="60.96" y2="8.255" width="0.254" layer="1"/>
 <contactref element="SW1X11" pad="6"/>
 <contactref element="IC1X11" pad="17"/>
@@
 </signal>
 <signal name="N$1X11">
-<wire x1="47.21" y1="27.94" x2="47.21" y2="27.994" width="0.4064" layer="1"/>
-<wire x1="47.21" y1="27.994" x2="45.046" y2="27.94" width="0.4064" layer="1"/>
+<wire x1="47.51" y1="27.94" x2="47.21" y2="27.994" width="0.4064" layer="1"/>
+<wire x1="47.21" y1="27.994" x2="45.085" y2="27.94" width="0.4064" layer="1"/>
 <contactref element="R4X11" pad="1"/>
 <contactref element="LED1X11" pad="A"/>
@@
 <wire x1="50.8" y1="14.605" x2="50.165" y2="15.24" width="0.254" layer="1"/>
 <wire x1="50.165" y1="15.24" x2="50.165" y2="27.085" width="0.254" layer="1"/>
-<wire x1="50.165" y1="27.085" x2="49.31" y2="27.94" width="0.254" layer="1"/>
+<wire x1="50.165" y1="27.085" x2="49.01" y2="27.94" width="0.254" layer="1"/>
 <contactref element="IC1X11" pad="20"/>
 <contactref element="LED1X11" pad="C"/>
@@
 <signal name="A0X12">
 <wire x1="52.278" y1="41.275" x2="55.88" y2="41.275" width="0.254" layer="1"/>
-<wire x1="57.15" y1="40.22" x2="55.88" y2="41.275" width="0.254" layer="1"/>
+<wire x1="57.15" y1="40.259" x2="55.88" y2="41.275" width="0.254" layer="1"/>
 <wire x1="59.69" y1="38.735" x2="73.66" y2="38.735" width="0.254" layer="1"/>
 <wire x1="73.66" y1="38.735" x2="76.2" y2="41.275" width="0.254" layer="1"/>
@@
 <wire x1="59.69" y1="38.735" x2="58.42" y2="40.005" width="0.254" layer="1"/>
 <wire x1="58.42" y1="40.005" x2="57.365" y2="40.005" width="0.254" layer="1"/>
-<wire x1="57.365" y1="40.005" x2="57.15" y2="40.22" width="0.254" layer="1"/>
+<wire x1="57.365" y1="40.005" x2="57.15" y2="40.259" width="0.254" layer="1"/>
 <contactref element="SW1X12" pad="8"/>
 <contactref element="IC1X12" pad="15"/>
@@
 <wire x1="72.39" y1="40.005" x2="73.66" y2="41.275" width="0.254" layer="1"/>
 <wire x1="73.66" y1="41.275" x2="73.66" y2="44.45" width="0.254" layer="1"/>
-<wire x1="64.135" y1="42.965" x2="65.19" y2="42.965" width="0.254" layer="1"/>
+<wire x1="64.135" y1="42.926" x2="65.19" y2="42.965" width="0.254" layer="1"/>
 <wire x1="65.19" y1="42.965" x2="67.31" y2="45.085" width="0.254" layer="1"/>
 <wire x1="67.31" y1="45.085" x2="73.025" y2="45.085" width="0.254" layer="1"/>
@@
 <wire x1="69.85" y1="41.275" x2="71.12" y2="42.545" width="0.254" layer="1"/>
 <wire x1="71.12" y1="42.545" x2="71.12" y2="43.18" width="0.254" layer="1"/>
-<wire x1="60.96" y1="42.965" x2="60.96" y2="41.275" width="0.254" layer="1"/>
+<wire x1="60.96" y1="42.926" x2="60.96" y2="41.275" width="0.254" layer="1"/>
 <contactref element="SW1X12" pad="6"/>
 <contactref element="IC1X12" pad="17"/>
@@
 </signal>
 <signal name="N$1X12">
-<wire x1="47.21" y1="60.96" x2="47.21" y2="61.014" width="0.4064" layer="1"/>
-<wire x1="47.21" y1="61.014" x2="45.046" y2="60.96" width="0.4064" layer="1"/>
+<wire x1="47.51" y1="60.96" x2="47.21" y2="61.014" width="0.4064" layer="1"/>
+<wire x1="47.21" y1="61.014" x2="45.085" y2="60.96" width="0.4064" layer="1"/>
 <contactref element="R4X12" pad="1"/>
 <contactref element="LED1X12" pad="A"/>
@@
 <wire x1="50.8" y1="47.625" x2="50.165" y2="48.26" width="0.254" layer="1"/>
 <wire x1="50.165" y1="48.26" x2="50.165" y2="60.105" width="0.254" layer="1"/>
-<wire x1="50.165" y1="60.105" x2="49.31" y2="60.96" width="0.254" layer="1"/>
+<wire x1="50.165" y1="60.105" x2="49.01" y2="60.96" width="0.254" layer="1"/>
 <contactref element="IC1X12" pad="20"/>
 <contactref element="LED1X12" pad="C"/>
@@
 <signal name="A0X13">
 <wire x1="52.278" y1="74.295" x2="55.88" y2="74.295" width="0.254" layer="1"/>
-<wire x1="57.15" y1="73.24" x2="55.88" y2="74.295" width="0.254" layer="1"/>
+<wire x1="57.15" y1="73.279" x2="55.88" y2="74.295" width="0.254" layer="1"/>
 <wire x1="59.69" y1="71.755" x2="73.66" y2="71.755" width="0.254" layer="1"/>
 <wire x1="73.66" y1="71.755" x2="76.2" y2="74.295" width="0.254" layer="1"/>
@@
 <wire x1="59.69" y1="71.755" x2="58.42" y2="73.025" width="0.254" layer="1"/>
 <wire x1="58.42" y1="73.025" x2="57.365" y2="73.025" width="0.254" layer="1"/>
-<wire x1="57.365" y1="73.025" x2="57.15" y2="73.24" width="0.254" layer="1"/>
+<wire x1="57.365" y1="73.025" x2="57.15" y2="73.279" width="0.254" layer="1"/>
 <contactref element="SW1X13" pad="8"/>
 <contactref element="IC1X13" pad="15"/>
@@
 <wire x1="72.39" y1="73.025" x2="73.66" y2="74.295" width="0.254" layer="1"/>
 <wire x1="73.66" y1="74.295" x2="73.66" y2="77.47" width="0.254" layer="1"/>
-<wire x1="64.135" y1="75.985" x2="65.19" y2="75.985" width="0.254" layer="1"/>
+<wire x1="64.135" y1="75.946" x2="65.19" y2="75.985" width="0.254" layer="1"/>
 <wire x1="65.19" y1="75.985" x2="67.31" y2="78.105" width="0.254" layer="1"/>
 <wire x1="67.31" y1="78.105" x2="73.025" y2="78.105" width="0.254" layer="1"/>
@@
 <wire x1="69.85" y1="74.295" x2="71.12" y2="75.565" width="0.254" layer="1"/>
 <wire x1="71.12" y1="75.565" x2="71.12" y2="76.2" width="0.254" layer="1"/>
-<wire x1="60.96" y1="75.985" x2="60.96" y2="74.295" width="0.254" layer="1"/>
+<wire x1="60.96" y1="75.946" x2="60.96" y2="74.295" width="0.254" layer="1"/>
 <contactref element="SW1X13" pad="6"/>
 <contactref element="IC1X13" pad="17"/>
@@
 </signal>
 <signal name="N$1X13">
-<wire x1="47.21" y1="93.98" x2="47.21" y2="94.034" width="0.4064" layer="1"/>
-<wire x1="47.21" y1="94.034" x2="45.046" y2="93.98" width="0.4064" layer="1"/>
+<wire x1="47.51" y1="93.98" x2="47.21" y2="94.034" width="0.4064" layer="1"/>
+<wire x1="47.21" y1="94.034" x2="45.085" y2="93.98" width="0.4064" layer="1"/>
 <contactref element="R4X13" pad="1"/>
 <contactref element="LED1X13" pad="A"/>
@@
 <wire x1="50.8" y1="80.645" x2="50.165" y2="81.28" width="0.254" layer="1"/>
 <wire x1="50.165" y1="81.28" x2="50.165" y2="93.125" width="0.254" layer="1"/>
-<wire x1="50.165" y1="93.125" x2="49.31" y2="93.98" width="0.254" layer="1"/>
+<wire x1="50.165" y1="93.125" x2="49.01" y2="93.98" width="0.254" layer="1"/>
 <contactref element="IC1X13" pad="20"/>
 <contactref element="LED1X13" pad="C"/>
